File: kicad/A1.kicad_sch (KiCad schematic)
At the start: 108 parts, among them IC1 LM1458, IC2 LM741, IC3 LM741, J206 J206, P1 P1, P2 P2, P3 P3, Q1 2N3054, Q2 2N3053, Q3 2N3053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

Commit message: Redone A1.
Parts:
- removed unit 6 of J206
- removed unit 3 of J206
- removed unit 4 of J206
- removed unit 1 of J206
- removed unit 10 of J206
- removed unit 5 of J206
- removed unit 11 of J206
- removed unit 9 of J206
- removed unit 18 of J206
- removed unit 15 of P1
- removed unit 13 of P1
- added C202: 10mF, symbol Elektuur:C-polar
- added CR201, CR202: D, symbol Elektuur:D
- added F202: 6AS, symbol Elektuur:F
- added J? (x8): J-terminal, symbol Elektuur:J-terminal
- added unit 15 of P1
- added unit 13 of P1
- added unit 17 of P1
- added Q401, Q501: 2N3054, symbol Elektuur:T-BJT-NPN
- added R201: 220, symbol Elektuur:R
- added T201, T201_2: L, symbol Elektuur:L
- CR102: value Th -> IR30A
- CR103: value D -> 40HF10
- P1: symbol Elektuur:J-terminal-18 -> Elektuur:J-terminal-thru-18
- P2: symbol Elektuur:J-terminal-3 -> Elektuur:J-terminal-thru-3
- R102: Spice_Model lin100k -> lin10k
- R103: Spice_Model lin100k -> lin7k
Connections:
- net TOP+ is gone; now on net +ISENSE: R3.1 (+), R4.1 (+), R7.1 (+)
- net (-): now also R46.1 (+); no longer R46.2 (-)
- net -S: now also R19.1 (+), R29.2 (-); no longer R19.2 (-), R29.1 (+)
- net 0: now also P1.18
- net S102:12: now reaches P1.16
- net S102:12: no longer R19.1 (+)
- net at R102.3 (c): now also P1.6
- net -ISENSE: now reaches C8.1 (+), QD4.1, R24.2 (-), R25.1 (+), TB1.2
- net -ISENSE: now also R27.2 (-), P1.13; no longer R27.1 (+)
- net at IC2.3 (+): now also R29.1 (+); no longer R29.2 (-)
- net at C11.1 (+): now also R46.2 (-); no longer R46.1 (+)
- net at IC1.6 (-), R20.1 (+), R23.2 (-): now also R15.2 (-); no longer R15.1 (+)
- net at DS101.1 (K-): now also P1.3
- net at IC1.3 (+): now also R27.1 (+); no longer R27.2 (-)
- net at QD2.1: now also J?.1; no longer R12.1 (+)
- net at CR9.1 (K-): now also R16.1 (+); no longer R16.2 (-)
- net at P1.11: now also R28.2 (-); no longer R28.1 (+)
- net at R102.2 (b): now also P1.4
- net at DS101.2 (A+): now also P1.1
- net at C4.1 (+): now also IC1.7 (OUTB), R16.2 (-); no longer R15.2 (-)
- net at R102.1 (a): now also P1.5
- net at R22.2 (-): now also IC1.1 (OUTA), R21.1 (+); no longer IC1.5 (+)
- net IND: now reaches CR14.1 (K-), CR17.2 (A+), P1.3, R43.1 (+)
- net at R103.3 (c): now also P1.10
- net at C5.1 (+): now also IC2.6 (OUT), R33.2 (-); no longer R31.2 (-)
- net at QD5.2: now also J?.1, R201.2 (-), T201.2 (-), T201_2.1 (+)
- net at R103.1 (a): now also P1.9
- net at R103.2 (b): now also P1.11
- net at QD2.2: now also R12.2 (-)
- net at QD1.1: now also J?.1; no longer R13.1 (+)
- net at CR13.1 (K-): now also R33.1 (+); no longer R33.2 (-)
- net at QD1.2: now also R13.2 (-)
- net +TOP renamed +ISENSE
- net +ISENSE: now also R12.1 (+), R13.1 (+), R26.2 (-), P1.15; no longer R12.2 (-), R13.2 (-), R26.1 (+)
- new net: J?.1, P1.7
- new net: P1.16, R19.2 (-)
- new net: J?.1, Q401.1 (C)
- new net: J?.2, Q401.2 (B)
- new net: J?.2, Q401.3 (E)
- new net: CR202.2 (A+), P2.2, T201_2.2 (-)
- new net: CR201.1 (K-), CR202.1 (K-), F202.2 (-), J?.2, R201.1 (+)
- new net: CR201.2 (A+), P2.1, T201.1 (+)
- new net: J?.1, P1.8
- new net: J?.2, Q501.3 (E)
- new net: IC1.2 (-), R21.2 (-), R26.1 (+)
- new net: C4.2 (-), R15.1 (+)
- new net: F202.1 (+), J?.2, J?.2, P2.3
- new net: IC1.5 (+), R22.1 (+)
- new net: J?.1, Q501.1 (C)
- new net: J?.2, Q501.2 (B)
- new net: C5.2 (-), R31.1 (+)
- new net: IC2.2 (-), R28.1 (+), R31.2 (-)
- new net: C202.1 (+), J?.1
- new net: C202.2 (-), J?.2
- new net S102:3: P1.14 (e14)
- new net S102:6: P1.15
- new net S102:9: P1.13
- no-connect marks 3 -> 2
Other:
- note added: "0-6V VOLTAGE CONTROL"
- note added: "3xRD"
- note added: "AUX SCR"
- note added: "BK/WH"
- note added: "BK/YE"
- note added: "BN"
- note added: "BU"
- note added: "CROWBAR"
- note added: "CROWBAR LEVEL CONTROL 4-8V"
- note added: "FRONT PANEL"
- note added: "G=-10"
- note added: "I_{O} REGULATOR"
- note added: "I_{O} SENSE AMP"
- note added: "J206"
- note added: "J207"
- note added: "J21"
- note added: "J22"
- note added: "J26"
- note added: "J27"
- note added: "PASS ELEMENTS"
- note added: "REFERENCE"
- note added: "SCR DRIVER"
- note added: "THICK"
- note added: "THIN"
- note added: "TRANSFORMER SECONDARY"
- note added: "VT"
- note added: "WH"
- note added: "WH/BN"
- note added: "WH/BU"
- note added: "YE"
- note removed: "**"
- note removed: "BK/WH THIN"
- note removed: "BRN"
- note removed: "CROWBAR LEVEL SET 4-8V"
- note removed: "FRONT TERMINALS"
- note removed: "I REGULATOR"
- note removed: "I_{O} SENSE G=-10"
- note removed: "PASS TRANSISTOR DRIVE OUTPUT"
- note removed: "VIOL"
- note removed: "WH/BLU"
- note removed: "WH/BRN"
- note removed: "YEL"
- company: KEPCO -> A design by KEPCO
- title: MPS620M A1: 6V, 6A Supply Assy -> MPS620M A1: 6V, 5A Supply Assy 235-0690
- moved on the sheet: BP104, BP105, BP106, BP107, BP108, C1, C10, C11, C2, C3, C4, C5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

Commit message: Tweak A1 BOM & legends.
Parts:
- C202: Rating 20V -> V
- C4, C5: Rating V -> 200V
- C6: Rating V -> 500V
- CR1, CR2: value D -> DR; Rating V/A -> 100V, 1.5A
- CR10: value 6.2V -> 6.2V 5%; Rating W -> 7.5mA
- CR13, CR14, CR15, CR6, CR9: value D -> DSW; Rating V/A -> 75V, 0.4W
- CR16: value 3.3V -> 3.3V 1N746A; Rating W -> 0.4W
- CR17: value Th -> S2061Y
- CR5: Rating W -> 0.5W
- CR7, CR8: value 1N963B -> 12V 1N963B; Rating W -> 10mA
- DS101: Rating 20mA -> A
- R1: Rating W -> 3W
- R10, R18: Rating 1% -> 1/2W
- R102: Spice_Model lin10k -> lin100k
- R11, R45, R9: Rating W -> 1W
- R12, R13, R24: Rating W -> 5W
- R17, R43, R44, R7, R8: Rating W -> 1/2W
- R19, R20, R21, R23, R26, R31, R32, R34, R37, R38, R40: Rating 1% -> W
- R2: value 2k0 -> 2k; Rating W -> 1/2W
- R41: value 1k0 -> 1k
Other:
- note added: "CROWBAR LEVEL CONTROL 2.7-6.2V"
- note added: "I_{O} LIMIT AMP"
- note added: "bleeder"
- note added: "load equalization"
- note removed: "CROWBAR LEVEL CONTROL 4-8V"
- note removed: "I_{O} LIMIT"
- note removed: "I_{O} REGULATOR"
- moved on the sheet: R17, R2, R3, R5, R6, R7

Commit message: Done A1, A3.
Parts:
- BP104: Label (none) -> G
- BP105: Label (none) -> -S
- BP106: Label (none) -> -
- BP107: Label (none) -> +
- BP108: Label (none) -> +S
- C202: Rating V -> 20V
- CR201, CR202: value D -> R2010; Rating V/A -> 100V, 16A
- F202: value 6AS -> 6AS MTH
- R103: value 7k -> 7.0k
- R16, R22, R23, R26, R27, R28, R29, R33, R41, R42, R43: value 1k -> 1.0k
- R201: Rating W -> 2W
- R32: value 2k0 -> 2.0k
- gave numbers to parts that had none: 8
- renumbered CR3_01 to CR3_1, CR3_02 to CR3_2, CR3_03 to CR3_3, CR4_01 to CR4_1, CR4_02 to CR4_2, CR4_03 to CR4_3
Other:
- note added: "A1"
- note added: "A2"
- note added: "A4"
- note added: "A5"
- note added: "CC LOAD"
- note added: "LOAD EQUALIZATION"
- note added: "P.O."
- note added: "XFMR SEC."
- note removed: "(+)"
- note removed: "(+S)"
- note removed: "(-)"
- note removed: "(-S)"
- note removed: "(GROUND)"
- note removed: "TRANSFORMER SECONDARY"
- note removed: "load equalization"
- moved on the sheet: BP104, BP105, BP106, BP107, BP108, IC1C, IC2B, Q401
