File: kicad/A3.kicad_sch (KiCad schematic)
At the start: 0 parts

Commit message: WIP A3.
Parts:
- added BP? (x5): K-socket-1, symbol Elektuur:K-socket-1
- added C301, C303: 1500u, symbol Elektuur:C-polar
- added C?: 0.01u, symbol Elektuur:C
- added C?: 0.1u, symbol Elektuur:C
- added C?: 100p, symbol Elektuur:C
- added C?: 950u, symbol Elektuur:C-polar
- added C?: 1n, symbol Elektuur:C
- added C?: 1000u, symbol Elektuur:C-polar
- added C? (x3): 150u, symbol Elektuur:C-polar
- added C?: 10mF, symbol Elektuur:C-polar
- added C?: 110u, symbol Elektuur:C-polar
- added C?: 22u, symbol Elektuur:C-polar
- added CR301, CR302, CR303, CR304, CR311, CR312, CR313, CR314, CR3_? (x3), CR?: D-45, symbol Elektuur:D-45
- added CR305, CR306, CR315, CR316, CR328, CR330, CR331, CR332, CR? (x8): D, symbol Elektuur:D
- added CR?: 6.2V, symbol Elektuur:D-Zener
- added CR? (x2): 1N963B, symbol Elektuur:D-Zener
- added CR?: 6.8V, symbol Elektuur:D-Zener
- added CR?: 3.3V, symbol Elektuur:D-Zener
- added CR?: 40HF10, symbol Elektuur:D
- added CR?: HVP, symbol Elektuur:D
- added CR?: Th, symbol Elektuur:Th
- added CR?: IR30A, symbol Elektuur:Th
- added CX? (x2): DNP, symbol Elektuur:C
- added DS?: 1.8V, symbol Elektuur:D-LED
- added F?: 6AS, symbol Elektuur:F
- added IC? (x3): LM1458, symbol Elektuur:A-opamp-dual
- added IC? (x5): LM741, symbol Elektuur:A-opamp
- added J? (x8), QD? (x7): J-terminal, symbol Elektuur:J-terminal
- added J?: J206, symbol Elektuur:J-terminal-18
- added P301: P301, symbol Elektuur:J-terminal-thru-6
- added P305, P?: P305, symbol Elektuur:J-terminal-thru-22
- added P? (x16): P1, symbol Elektuur:J-terminal-thru-18
- added P? (x3): P2, symbol Elektuur:J-terminal-thru-3
- added P?: P1, symbol Elektuur:J-terminal-18
- added P? (x4): P3, symbol Elektuur:J-terminal-5
- added Q301, Q? (x2): 2N3053, symbol Elektuur:T-BJT-NPN
- added Q303: 2N4036, symbol Elektuur:T-BJT-PNP
- added Q? (x3): 2N3054, symbol Elektuur:T-BJT-NPN
- added Q?: 2N4355, symbol Elektuur:T-BJT-PNP
- added R301, R311: 39, symbol Elektuur:R
- added R302, R312: 2k, symbol Elektuur:R
- added R304, R315, R?: 500, symbol Elektuur:R
- added R305, R313, R? (x8): 1k, symbol Elektuur:R
- added R306, R316: 0.5, symbol Elektuur:R
- added R? (x2): 10k, symbol Elektuur:R
- added R? (x2): 8.06k, symbol Elektuur:R
- added R?: 1k0, symbol Elektuur:R
- added R? (x4): 10, symbol Elektuur:R
- added R? (x2): 220, symbol Elektuur:R
- added R?: 2.74k, symbol Elektuur:R
- added R? (x2): 560, symbol Elektuur:R
- added R?: 7k, symbol Elektuur:P
- added R?: 1.2k, symbol Elektuur:R
- added R?: 2.2k, symbol Elektuur:R
- added R? (x2): 2k0, symbol Elektuur:R
- added R?: 82k, symbol Elektuur:R
- added R?: 137, symbol Elektuur:R
- added R?: 470, symbol Elektuur:R
- added R?: 2.7k, symbol Elektuur:R
- added R? (x2): 0.2, symbol Elektuur:R
- added R? (x3): 100, symbol Elektuur:R
- added R?: 8.66k, symbol Elektuur:R
- added R? (x2): 6.98k, symbol Elektuur:R
- added R?: 390, symbol Elektuur:R
- added R?: 0.1, symbol Elektuur:R
- added R?: 1.5k, symbol Elektuur:R
- added R?: 10k, symbol Elektuur:P
- added R?: 619, symbol Elektuur:R
- added T201_?, T?: L, symbol Elektuur:L
- added TB? (x5): TB1, symbol Elektuur:J-terminal-5
Connections:
- new net: P?.6, R?.1 (+)
- new net: CR332.2 (A+), Q303.1 (C), R313.1 (+)
- new net: Q303.3 (E), R311.2 (-), R313.2 (-)
- new net: CR305.2 (A+), CR328.2 (A+), P305.4, Q301.2 (B), R302.2 (-), R304.1 (+)
- new net: CR331.2 (A+), P305.13, P305.14 (e14), R304.2 (-), R306.1 (+)
- new net: CR?.1 (K-), Q?.2 (B), R?.2 (-)
- new net: CX?.2 (-), Q?.3 (E), R?.1 (+), R?.2 (-), R?.2 (-)
- new net: CR311.1 (K-), CR314.2 (A+), P301.5
- new net: C303.2 (-), CR311.2 (A+), CR312.2 (A+), P305.7, R312.1 (+)
- new net: DS?.1 (K-), P?.3
- new net: CR?.1 (K-), CR?.1 (K-), F?.2 (-), J?.2, R?.1 (+)
- new net: CR?.2 (A+), P?.2, T201_?.2 (-)
- new net: CR316.1 (K-), CR330.1 (K-), P305.3, Q303.2 (B), R312.2 (-), R315.1 (+)
- new net: CR332.1 (K-), P305.12, P?.11, R315.2 (-), R316.2 (-)
- new net: DS?.2 (A+), P?.1
- new net: J?.1, P?.7
- new net: J?.2, Q?.2 (B) (x2)
- new net: C?.1 (+), IC?.7 (OUTB)
- new net: C?.2 (-), R?.1 (+) (x2)
- new net: C301.2 (-), CR301.2 (A+), CR303.2 (A+), CR306.1 (K-), R301.1 (+)
- new net: CR305.1 (K-), CR306.2 (A+)
- new net: CR331.1 (K-), Q301.1 (C), R305.2 (-)
- new net: CR?.2 (A+), CR?.3 (G), R?.2 (-)
- new net: CR?.1 (K-), P?.2
- new net: C?.1 (+), R?.2 (-)
- new net: CR?.1 (K-), P?.1
- new net: CR303.1 (K-), CR304.2 (A+), P301.4
- new net: CR3_?.1 (K-), CR3_?.2 (A+), P?.2
- new net: Q?.1 (C), R?.2 (-)
- new net: C?.2 (-), IC?.2 (-), R?.1 (+), R?.2 (-)
- new net: IC?.3 (+), P?.4
- new net: CR?.2 (A+), IC?.6 (OUT)
- new net: J?.1, P?.8
- new net: P?.7, P?.8, Q?.3 (E), R?.2 (-), R?.2 (-)
- new net: CR?.2 (A+), P?.1, T?.1 (+)
- new net: J?.1, QD?.1 (x2)
- new net: J?.2, Q?.3 (E) (x2)
- new net: C?.2 (-), P?.18, TB?.3
- new net: QD?.2, R?.2 (-) (x2)
- new net: IC?.2 (-), R?.1 (+), R?.2 (-) (x2)
- new net: P?.11, R?.2 (-)
- new net: J?.1, Q?.1 (C) (x2)
- new net: IC?.3 (+), R?.1 (+) (x2)
- new net: C303.1 (+), CR313.1 (K-), CR314.1 (K-), CR315.2 (A+), R311.1 (+)
- new net: P?.10, R?.3 (c)
- new net: C?.2 (-), CR?.2 (A+), R?.2 (-)
- new net: Q?.1 (C), R?.1 (+), R?.2 (-)
- new net: CR?.1 (K-), R?.1 (+)
- new net: C?.1 (+), IC?.6 (OUT), R?.2 (-)
- new net: CR?.1 (K-), CR?.1 (K-)
- new net: P?.9, R?.1 (a)
- new net: P?.11, R?.2 (b)
- new net: Q301.3 (E), R301.2 (-), R305.1 (+)
- new net: Q?.2 (B), Q?.3 (E), R?.1 (+), R?.2 (-), R?.2 (-)
- new net: Q?.2 (B), R?.2 (-)
- new net: CR328.1 (K-), CR330.2 (A+), P305.10, P305.8, P305.9, R306.2 (-), R316.1 (+)
- new net: CR315.1 (K-), CR316.2 (A+)
- new net: CR?.1 (K-), CR?.2 (A+), QD?.2, R?.1 (+)
- new net: CR?.1 (K-), CR?.2 (A+), CR?.2 (A+), QD?.2
- new net: P?.6, R?.3 (c)
- new net: CR3_?.1 (K-), CR?.2 (A+), P?.1
- new net: CR301.1 (K-), CR302.2 (A+), P301.3
- new net: IC?.1 (OUTA), R?.1 (+), R?.2 (-)
- new net: IC?.6 (-), R?.1 (+), R?.2 (-), R?.2 (-)
- new net: F?.1 (+), J?.2, J?.2, P?.3
- new net: C301.1 (+), CR302.1 (K-), CR304.1 (K-), P305.22, R302.1 (+)
- new net: IC?.5 (OFSB), R?.1 (+)
- new net: IC?.1 (OFSA), R?.1 (+)
- new net: J?.1, QD?.2, R?.2 (-), T201_?.1 (+), T?.2 (-)
- new net: CR?.1 (K-), QD?.2
- new net: CR312.1 (K-), CR313.2 (A+), P301.6
- new net: CR?.3 (G), J?.2, R?.2 (-)
- new net: C?.2 (-), J?.2
- new net: IC?.5 (+), R?.1 (+)
- new net: P?.5, R?.1 (a)
- new net: C?.1 (+), J?.1
- new net: Q?.2 (B), R?.1 (+), R?.2 (-)
- new net: P?.4, R?.2 (b)
- new net: C?.1 (+), IC?.7 (+), R?.1 (+)
- new net: P?.3, Q?.1 (C)
- new net: CX?.1 (+), P?.4
- new net: CX?.2 (-), P?.3
- new net: P?.16, R?.2 (-)
- new net (-): C?.2 (-), C?.2 (-), QD?.1, QD?.1, R?.1 (+), R?.2 (-), TB?.4
- new net +12: C?.1 (+), CR?.1 (K-), IC?.7 (+), IC?.8 (+), R?.1 (+), R?.1 (+), R?.1 (+), R?.2 (-), R?.2 (-)
- new net +ISENSE: C?.2 (-), CR3_?.2 (A+), CR3_?.2 (A+), P?.15, R?.1 (+), R?.1 (+), R?.1 (+), R?.1 (+), R?.1 (+), R?.1 (+), R?.2 (-)
- new net -12: CR?.2 (A+), CX?.1 (+), IC?.4 (-), IC?.4 (-), IC?.4 (-), Q?.1 (C), R?.1 (+), R?.2 (-), R?.2 (-), R?.2 (-)
- new net -ISENSE: C?.1 (+), P?.13, QD?.1, R?.1 (+), R?.2 (-), R?.2 (-), TB?.2
- new net -S: C?.1 (+), C?.1 (+), C?.2 (-), QD?.1, R?.1 (+), R?.1 (+), R?.2 (-), TB?.5
- new net 0: C?.1 (+), C?.2 (-), C?.2 (-), CR?.1 (K-), CR?.1 (K-), CR?.1 (K-), CR?.2 (A+), P?.10, P?.14 (e14), P?.18, QD?.1, R?.1 (+), R?.2 (-), R?.2 (-), R?.2 (-), R?.2 (-), TB?.1
- new net EREF: CR?.2 (A+), P?.5, P?.9, R?.1 (+), R?.1 (+)
- new net GATE: CR?.2 (A+), CR?.2 (A+), CR?.2 (A+), R?.1 (+)
- new net IND: CR?.1 (K-), CR?.2 (A+), P?.3
- new net S102:12: P?.16
- new net S102:3: P?.14 (e14)
- new net S102:6: P?.15
- new net S102:9: P?.13
- new net SCR.DRIVE: P?.2, R?.1 (+)
- new net SCR.TRIG: P?.1, R?.1 (+)
- new net VDRV: C?.1 (+), CR3_?.1 (K-), CR?.1 (K-), Q?.3 (E), R?.2 (-), R?.2 (-)
- new net VRET: C?.1 (+), CR?.2 (A+), CR?.2 (A+), R?.1 (+), R?.1 (+)
- no-connect marks 0 -> 2
Other:
- note added: "(+)"
- note added: "(+S)"
- note added: "(-)"
- note added: "(-S)"
- note added: "(GROUND)"
- note added: "*"
- note added: "+S"
- note added: "-5.4V"
- note added: "-6.2V"
- note added: "0-6V VOLTAGE CONTROL"
- note added: "3xRD"
- note added: "AMPLIFIER SUPPLY"
- note added: "AUX SCR"
- note added: "BK"
- note added: "BK/WH"
- note added: "BK/WH THICK"
- note added: "BK/YE"
- note added: "BRN"
- note added: "BU"
- note added: "CHASSIS"
- note added: "CROWBAR"
- note added: "CROWBAR DETECTOR"
- note added: "CROWBAR LEVEL CONTROL 4-8V"
- note added: "FRONT PANEL"
- note added: "FRONT VOLTAGE CONTROLS"
- note added: "G=-10"
- note added: "GN"
- note added: "I_{O} LIMIT"
- note added: "I_{O} REGULATOR"
- note added: "I_{O} SENSE AMP"
- note added: "J206"
- note added: "J207"
- note added: "J21"
- note added: "J22"
- note added: "J23"
- note added: "J24"
- note added: "J25"
- note added: "J26"
- note added: "J27"
- note added: "PASS ELEMENTS"
- note added: "PRE-DRIVER"
- note added: "PRE-DRIVER SUPPLY"
- note added: "RD"
- note added: "RD/WH"
- note added: "REFERENCE"
- note added: "SCR DRIVER"
- note added: "TB1:+O"
- note added: "TB1:+S"
- note added: "TB1:-O"
- note added: "TB1:-S"
- note added: "TB1:GND"
- note added: "THICK"
- note added: "THIN"
- note added: "TRANSFORMER SECONDARY"
- note added: "V REGULATOR"
- note added: "VT"
- note added: "WH"
- note added: "WH/BK"
- note added: "WH/BRN"
- note added: "WH/BU"
- note added: "WH/PK"
- note added: "WH/RD"
- note added: "YE"
- note added: "YEL"
- company: KEPCO -> A design by KEPCO
- title: MPS620M A3: ±20V, 1A Supply Assy -> MPS620M A3: ±20V, 1A Supply Assy 236-0678

Commit message: WIP A3.
Parts:
- added BP101, BP102: K-socket-1, symbol Elektuur:K-socket-1
- added C304, C309: 0.1u, symbol Elektuur:C
- added C305, C308: 1n, symbol Elektuur:C
- added C306: 10n, symbol Elektuur:C
- added C311, C312: F, symbol Elektuur:C-polar
- added CR317, CR318 (x2), CR320, CR321, CR325, CR327: D, symbol Elektuur:D
- added CR322, CR328: 12V, symbol Elektuur:D-Zener
- added IC301: LM1458, symbol Elektuur:A-opamp-dual
- added unit 1 of IC302
- added unit 5 of P305
- added unit 20 of P305
- added P? (x4): P305, symbol Elektuur:J-terminal-thru-22
- added R317, R318, R352: 20k, symbol Elektuur:R
- added R318 (x2), R320, R329, R331, R337, R338, R348: 1k, symbol Elektuur:R
- added R321, R328, R347: 10, symbol Elektuur:R
- added R323, R327, R344: 220, symbol Elektuur:R
- added R325, R342: 2.4k, symbol Elektuur:R
- added R334: 960, symbol Elektuur:R
- added TB? (x2): TB301, symbol Elektuur:J-terminal-5
- C307: renamed from C?; value 1n -> 10n
- CR324: renamed from CR?; value 3.3V -> 12V
- R333: renamed from R?; value 6.98k -> 1k
- R339: renamed from R?; Rating 1% -> W
- R340: renamed from R?; value 1k -> 220
- TB301: renamed from TB?; value TB1 -> TB301
- gave numbers to parts that had none: 6
Connections:
- net +12: now also R342.2 (-); no longer IC?.8 (+)
- net -12: now also R325.1 (+)
- net -S: no longer TB301.5
- net 0: now also CR324.1 (K-), CR317.2 (A+), CR318.1 (K-), CR322.2 (A+), CR328.1 (K-), IC302.3 (+); no longer R333.2 (-)
- net GATE: no longer CR326.2 (A+)
- net at R?.1 (+): now also IC303.3 (+), CR328.2 (A+), R318.1 (+); no longer P?.6
- net at CR305.2 (A+), CR328.2 (A+), P305.4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: now also TB301.1
- net at CR331.2 (A+), P305.13, P305.14 (e14)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: now also R337.2 (-)
- net at CR316.1 (K-), CR330.1 (K-), P305.3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: now also TB?.1
- net at CR332.1 (K-), P305.12, P?.11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: now also R329.2 (-)
- net at C?.1 (+): no longer IC302.7 (OUTB)
- net at CR?.3 (G), R?.2 (-): no longer CR324.2 (A+)
- net at P301.4: now also CR303.1 (K-), CR304.2 (A+)
- net at C?.2 (-), R?.1 (+), R?.2 (-): no longer IC303.2 (-)
- net at P?.4: now also R?.2 (b); no longer IC303.3 (+)
- net at IC303.6 (OUT): now also C308.1 (+), R344.2 (-); no longer CR?.2 (A+)
- net at IC?.2 (-), R?.1 (+): no longer R339.2 (-)
- net at C307.1 (+), R340.2 (-): now also IC302.7 (OUTB); no longer IC?.6 (OUT)
- net at CR?.1 (K-): no longer CR324.1 (K-)
- net at CR328.1 (K-), CR330.2 (A+), P305.10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: now also TB?.1
- net at R?.2 (-), R?.2 (-): no longer IC302.6 (-), R333.1 (+)
- net at IC302.5 (+): now also R338.2 (-); no longer R?.1 (+)
- net at P305.8: now also P?.19
- net S201:10: now reaches P305.4
- net S201:10: now also P?.6
- net S201:2: now reaches P305.3
- net S201:2: now also P305.5
- new net: C304.2 (-), C312.1 (+), P305.5, R318.2 (-)
- new net: C311.1 (+), C312.2 (-), P?.19, R320.2 (-)
- new net: IC303.2 (-), R347.2 (-), R348.1 (+)
- new net: P?.18, R348.2 (-)
- new net: CR317.1 (K-), CR318.2 (A+), IC301.3 (+), R318.1 (+)
- new net: C305.1 (+), IC301.1 (OUTA), R323.2 (-)
- new net: IC301.2 (-), R320.1 (+), R321.2 (-)
- new net: CR322.1 (K-), IC301.6 (-), R328.2 (-), R329.1 (+)
- new net: CR327.1 (K-), R344.1 (+)
- new net: CR325.2 (A+), CR326.2 (A+), CR327.2 (A+), R342.1 (+)
- new net: CR318.2 (A+), R323.1 (+)
- new net: C309.2 (-), C311.2 (-), P?.6, R317.2 (-), R352.2 (-)
- new net: C304.1 (+), R317.1 (+), R318.1 (+), R318.2 (-)
- new net: IC302.1 (OUTA), R334.2 (-), R338.1 (+)
- new net: CR324.2 (A+), IC302.6 (-), R337.1 (+), R339.2 (-)
- new net: CR318.1 (K-), CR320.1 (K-), CR321.1 (K-), R325.2 (-)
- new net: CR320.2 (A+), R327.1 (+)
- new net: CR325.1 (K-), P?.21
- new net: C309.1 (+), R318.2 (-), R352.1 (+)
- new net: C306.1 (+), IC301.7 (OUTB), R327.2 (-)
- new net: IC302.2 (-), R333.2 (-), R334.1 (+)
- new net: CR321.2 (A+), P305.20
- new net: C306.2 (-), R328.1 (+)
- new net: IC301.5 (+), R331.2 (-)
- new net: C308.2 (-), R347.1 (+)
- new net: C305.2 (-), R321.1 (+)
- new net I_{SET}: R331.1 (+), R333.1 (+)
Other:
- note added: "(0)"
- note added: "E_{0} SET"
- note added: "E_{O} MASTER"
- note added: "E_{O} SLAVE"
- note added: "I_{O} MASTER"
- note added: "I_{O} SLAVE"
- note added: "J205"
- note added: "TB301:+OUT"
- note added: "TB301:-OUT"
- note added: "TB301:COM"
- note added: "WH/OR"
- note added: "WH/YE"
- note added: "to A7"
- note removed: "TB1:-S"
- moved on the sheet: BP103, C301, C303, C307, CR301, CR302, CR303, CR304, CR305, CR306, CR311, CR312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

Commit message: WIP A3.
Parts:
- added unit 3 of IC301
- added J? (x3): J-terminal, symbol Elektuur:J-terminal
- added unit 16 of P305
- added R330: 21k, symbol Elektuur:R
- C301, C303, C?: Rating 50V -> V
- C304, C309: value 0.1u -> 0.2u
- C311, C312: value F -> 200u; Rating V -> 50V
- C?: Rating 600V -> V
- C? (x3): Rating 15V -> V
- C? (x2): Rating 20V -> V
- C?: Rating 3V -> V
- C?: Rating 25V -> V
- CR? (x2): value 1N963B -> 12V 1N963B
- DS?: Rating 20mA -> A
- Q601: renamed from Q?; value 2N3054 -> 2N6576
- Q701: renamed from Q?; value 2N3054 -> 2N6051; symbol Elektuur:T-BJT-NPN -> Elektuur:T-BJT-PNP
- R301, R311, R317, R318, R325, R342, R352, R? (x2): Rating W -> 1/2W
- R302, R304, R305, R306, R312, R313, R315, R316: Rating W -> 3W
- R333, R334, R345, R? (x6): Rating 1% -> W
- R346: renamed from R2k; Rating 1% -> W
- R351: renamed from R?; Rating 1% -> W
- R?: value 1k0 -> 1k
- R?: Spice_Model lin7k -> lin100k
- R? (x2): Rating 1% -> 1/2W
- R? (x2): Rating W -> 1W
- R? (x3): Rating W -> 5W
- R?: Rating 3W -> W
- R?: Spice_Model lin10k -> lin100k
- gave numbers to parts that had none: 2
- renumbered CR318 to CR319, R318 to R319, R318 to R353
Connections:
- net +12: now also IC301.8 (+)
- net -12: now also IC301.4 (-)
- net 0: now also C311.1 (+), C312.2 (-), IC302.8 (+), P?.19, R320.2 (-), R330.1 (+)
- net at CR328.2 (A+), IC303.3 (+), R353.1 (+): no longer R351.1 (+)
- net at P305.7: now also J?.1
- net at J?.1: now also P305.20; no longer P?.7
- net at J?.2: now also Q701.2 (B); no longer Q601.2 (B)
- net S102:7: now reaches P305.13
- net at P301.4: now also CR303.1 (K-), CR304.2 (A+)
- net at QD?.1: no longer J?.1
- net at J?.2: now also Q701.1 (C); no longer Q601.3 (E)
- net at J?.1: no longer Q701.1 (C)
- net at J?.2: no longer Q701.2 (B)
- net at Q701.3 (E): now also J?.1; no longer J?.2
- net S102:5: now reaches P?.11
- net at P?.6: now also R?.3 (c)
- net at P305.14 (e14): now also J?.1
- net at Q601.1 (C): now also J?.1; no longer J?.1
- net at F?.1 (+), J?.2, P?.3: no longer J?.2
- net at C309.1 (+), R352.1 (+), R353.2 (-): now also R351.1 (+)
- net at P305.20: now also CR321.2 (A+)
- net at P305.22: now also J?.2
- net at P305.12: now also J?.2
- net at P?.4: now also R?.2 (b)
- net at P?.21: now also J?.1
- net S102:4: now reaches P305.9
- net S102:8: now reaches P305.10
- net S201:10 renamed S102:10
- net S201:2 renamed S102:2
- new net: J?.2, Q601.2 (B)
- new net: J?.2, Q601.3 (E)
- new net: P305.16, R330.2 (-)
- new net S102:1,11: P305.16
Other:
- note added: "BU*"
- note added: "CI LOAD"
- note added: "GN*"
- note added: "OG"
- note added: "OG/BU"
- note added: "REF INVERTER"
- note added: "WH*"
- note added: "YE*"
- note added: "YE/BK"
- note removed: "to A7"
- moved on the sheet: BP101, BP102, BP103, C305, C306, C307, C308, C312, CR305, CR306, CR315, CR316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

Commit message: WIP A3.
Parts:
- removed P? (x2): P1, symbol Elektuur:J-terminal-thru-18
- removed P? (x2): P3, symbol Elektuur:J-terminal-5
- added CR307, CR307_1, CR307_2, CR4_?: D-45, symbol Elektuur:D-45
- added unit 2 of P301
- added unit 9 of P301
- added unit 8 of P301
- added unit 1 of P301
- added unit 7 of P301
- added unit 17 of P305
- added P?: P305, symbol Elektuur:J-terminal-thru-22
- added R338: 4.7k, symbol Elektuur:R
- added T202B, T202C: L, symbol Elektuur:L
- C302: renamed from C?; Rating V -> 50V
- P301: symbol Elektuur:J-terminal-thru-6 -> Elektuur:J-terminal-thru-9
- R101: renamed from R?; Spice_Model lin100k -> lin7k
- R335: renamed from R?; value 10k -> 1.5k; Spice_Model lin100k -> lin1.5k
- gave numbers to parts that had none: 12
Connections:
- net +12: now also CR307.1 (K-), CR307_1.1 (K-); no longer R?.2 (-)
- net -12: no longer IC?.4 (-)
- net 0: now also R335.3 (c), P305.17; no longer P?.10
- net EREF: no longer CR323.2 (A+), R332.1 (+)
- net I_{SET}: now also R335.2 (b)
- net E_{0 SET}: now reaches P?.18, R348.2 (-)
- net at P301.4: now also T202B.1 (+)
- net at CR?.2 (A+), P?.1: no longer T202A.1 (+)
- net at P?.10: no longer R101.3 (c)
- net at C302.2 (-), CR308.2 (A+), R309.2 (-): now also CR307_2.2 (A+), CR4_?.2 (A+)
- net at R101.1 (a): now also P?.15
- net at R101.2 (b): now also P?.18; no longer P?.11
- net at J?.1, QD?.2, R?.2 (-)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: no longer T202A.2 (-)
- net at P301.3: now also T202B.2 (-)
- net at R335.1 (a): now also R338.1 (+)
- net at P301.6: now also T202A.1 (+)
- net at P301.5: now also T202A.2 (-)
- net at CX?.1 (+): now also CR307.2 (A+), CR4_?.1 (K-), P301.9
- net at CX?.2 (-): now also CR307_1.2 (A+), CR307_2.1 (K-), P301.7
- new net: P301.7, T202C.1 (+)
- new net: P301.9, T202C.2 (-)
- new net: P305.17, R101.3 (c)
- new net REF: CR323.2 (A+), P?.15, R332.1 (+), R338.2 (-)
- now unconnected: P?.4, P?.6
- no-connect marks 2 -> 8
Other:
- note added: "BN"
- note added: "FRONT CONTROLS"
- note added: "GN/BK"
- note added: "J201"
- note added: "RD/BK"
- note removed: "E_{0} SET"
- note removed: "FRONT VOLTAGE CONTROLS"
- moved on the sheet: C302, CR308, CR309, CR310, CR323, Q302, R101, R307, R308, R309, R310, R332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

Commit message: Done A1, A3.
Parts:
- removed BP? (x4): K-socket-1, symbol Elektuur:K-socket-1
- removed C?: 0.01u, symbol Elektuur:C
- removed C?: 100p, symbol Elektuur:C
- removed C?: 950u, symbol Elektuur:C-polar
- removed C?: 1000u, symbol Elektuur:C-polar
- removed C? (x3): 150u, symbol Elektuur:C-polar
- removed C?: 10mF, symbol Elektuur:C-polar
- removed C?: 22u, symbol Elektuur:C-polar
- removed CR3_? (x3), CR?: D-45, symbol Elektuur:D-45
- removed CR? (x7): D, symbol Elektuur:D
- removed CR?: 40HF10, symbol Elektuur:D
- removed CR?: HVP, symbol Elektuur:D
- removed CR?: Th, symbol Elektuur:Th
- removed CR?: IR30A, symbol Elektuur:Th
- removed DS?: 1.8V, symbol Elektuur:D-LED
- removed F?: 6AS, symbol Elektuur:F
- removed IC?: LM1458, symbol Elektuur:A-opamp-dual
- removed IC? (x2): LM741, symbol Elektuur:A-opamp
- removed J? (x5), QD? (x7): J-terminal, symbol Elektuur:J-terminal
- removed J?: J206, symbol Elektuur:J-terminal-18
- removed P? (x14): P1, symbol Elektuur:J-terminal-thru-18
- removed P? (x3): P2, symbol Elektuur:J-terminal-thru-3
- removed P?: P1, symbol Elektuur:J-terminal-18
- removed P? (x2): P3, symbol Elektuur:J-terminal-5
- removed Q?: 2N3053, symbol Elektuur:T-BJT-NPN
- removed Q?: 2N4355, symbol Elektuur:T-BJT-PNP
- removed Q?: 2N3054, symbol Elektuur:T-BJT-NPN
- removed R? (x2): 10k, symbol Elektuur:R
- removed R? (x8): 1k, symbol Elektuur:R
- removed R? (x2): 220, symbol Elektuur:R
- removed R?: 2.74k, symbol Elektuur:R
- removed R? (x2): 560, symbol Elektuur:R
- removed R?: 2.2k, symbol Elektuur:R
- removed R? (x2): 10, symbol Elektuur:R
- removed R?: 470, symbol Elektuur:R
- removed R? (x2): 0.2, symbol Elektuur:R
- removed R? (x3): 100, symbol Elektuur:R
- removed R?: 8.66k, symbol Elektuur:R
- removed R?: 2k0, symbol Elektuur:R
- removed R?: 500, symbol Elektuur:R
- removed R?: 0.1, symbol Elektuur:R
- removed R?: 6.98k, symbol Elektuur:R
- removed R?: 1.5k, symbol Elektuur:R
- removed T201_?: L, symbol Elektuur:L
- removed TB? (x4): TB1, symbol Elektuur:J-terminal-5
- added unit 1 of P305
- added unit 2 of TB301
- BP101: Label (none) -> -
- BP102: Label (none) -> 0
- BP103: Label (none) -> +
- C301, C303: Rating V -> 75V
- C304, C305, C306, C307, C308, C309: Rating V -> 200V
- C310: renamed from C?; Rating V -> 600V
- CR301, CR302, CR303, CR304, CR311, CR312, CR313, CR314: value D-45 -> DR; Rating V/A -> 100V, 1.5A
- CR305, CR306, CR315, CR316, CR330: value D -> DR; Rating V/A -> 100V, 1.5A
- CR308: Rating W -> 0.5W
- CR322, CR324, CR328: value 12V -> 12V 1N963B
- CR323: value 6.2V -> 6.0V; Rating W -> 7.5mA
- CR329: renamed from CR328; value D -> DR; Rating V/A -> 100V, 1.5A
- CX301: renamed from CX?; now left out of the parts list
- R101: value 7k -> 7.0k
- R302, R312: value 2k -> 2.0k
- R305, R313, R319, R320, R329, R331, R333, R337, R338, R348, R353: value 1k -> 1.0k
- R336: renamed from R338; Rating W -> 1/2W
- R346: value 2k0 -> 2.0k
- TB301: renamed from TB?; symbol Elektuur:J-terminal-5 -> Elektuur:J-terminal-4
- TB301: symbol Elektuur:J-terminal-5 -> Elektuur:J-terminal-4
- gave numbers to parts that had none: 10
- renumbered T202A to T202A1, T202B to T202B1, T202C to T202C1
Connections:
- net (-) is gone; now on an unnamed net: R354.1 (+)
- net 0: now also R335.1 (a), P305.1; no longer R335.3 (c)
- net at R336.1 (+): now also R335.3 (c); no longer R335.1 (a)
- net at CR316.1 (K-), CR330.1 (K-), P305.3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: now also TB301.4; no longer TB301.1
- net at C310.2 (-): now also P305.1, TB301.2
- net at CR329.1 (K-), CR330.2 (A+), P305.10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: now also TB301.3; no longer TB301.1
- no-connect marks 8 -> 6
Other:
- note added: "A2"
- note added: "A3"
- note added: "A6"
- note added: "A7"
- note added: "CC LOAD"
- note added: "LOAD EQUALIZATION"
- note added: "P.O."
- note added: "TB301:GND"
- note removed: "(+)"
- note removed: "(+S)"
- note removed: "(-)"
- note removed: "(-S)"
- note removed: "(0)"
- note removed: "(GROUND)"
- note removed: "+S"
- note removed: "-5.4V"
- note removed: "-6.2V"
- note removed: "0-6V VOLTAGE CONTROL"
- note removed: "3xRD"
- note removed: "AUX SCR"
- note removed: "BK/WH"
- note removed: "BK/WH THICK"
- note removed: "BK/YE"
- note removed: "BRN"
- note removed: "CI LOAD"
- note removed: "CROWBAR"
- note removed: "CROWBAR DETECTOR"
- note removed: "CROWBAR LEVEL CONTROL 4-8V"
- note removed: "G=-10"
- note removed: "I_{O} LIMIT"
- note removed: "I_{O} REGULATOR"
- note removed: "I_{O} SENSE AMP"
- note removed: "J206"
- note removed: "J207"
- note removed: "J21"
- note removed: "J22"
- note removed: "J23"
- note removed: "J24"
- note removed: "J25"
- note removed: "J26"
- note removed: "J27"
- note removed: "PRE-DRIVER"
- note removed: "PRE-DRIVER SUPPLY"
- note removed: "RD/WH"
- note removed: "SCR DRIVER"
- note removed: "TB1:+O"
- note removed: "TB1:+S"
- note removed: "TB1:-O"
- note removed: "TB1:GND"
- note removed: "THICK"
- note removed: "THIN"
- note removed: "TRANSFORMER SECONDARY"
- note removed: "V REGULATOR"
- note removed: "WH/BRN"
- note removed: "WH/BU"
- note removed: "WH/PK"
- note removed: "WH/RD"
- note removed: "YEL"
- moved on the sheet: BP101, BP102, BP103, C301, C303, C310, CR305, CR306, CR315, CR316, CR329, CR330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
